File: hardware-rev1/ergogen/build/pcbs/slimdash_left.kicad_pcb (KiCad board)
At the start: 2 copper layers, 157.1 x 130 mm, 70 parts

Commit message: make initial left boards
Parts:
- moved D1 6.00 mm to (58.0, 97.0), turned to 270 degrees
- moved D10 6.00 mm to (96.0, 73.2), turned to 270 degrees
- moved D11 6.00 mm to (96.0, 54.1), turned to 270 degrees
- moved D12 6.00 mm to (96.0, 35.1), turned to 270 degrees
- moved D13 6.00 mm to (115.0, 89.9), turned to 270 degrees
- moved D14 6.00 mm to (115.0, 70.8), turned to 270 degrees
- moved D15 6.00 mm to (115.0, 51.8), turned to 270 degrees
- moved D16 6.00 mm to (115.0, 32.7), turned to 270 degrees
- moved D17 6.00 mm to (134.0, 92.2), turned to 270 degrees
- moved D18 6.00 mm to (134.0, 73.2), turned to 270 degrees
- moved D19 6.00 mm to (134.0, 54.1), turned to 270 degrees
- moved D2 6.00 mm to (58.0, 78.0), turned to 270 degrees
- moved D20 6.00 mm to (134.0, 35.1), turned to 270 degrees
- moved D21 6.00 mm to (153.0, 94.6), turned to 270 degrees
- moved D22 6.00 mm to (153.0, 75.6), turned to 270 degrees
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Other:
- board size 157.1 x 130 mm -> 157.1 x 131.5 mm
