File: hardware-rev1/ergogen/build/pcbs/slimdash.kicad_pcb (KiCad board)
At the start: 2 copper layers, 157.1 x 131.5 mm, 70 parts

Commit message: fix some positioning and net labels
Connections:
- net ROW5 renamed ROW0
- D1 pad 1: ROW2 -> ROW3
- D10 pad 1: ROW3 -> ROW2
- D11 pad 1: ROW4 -> ROW1
- D13 pad 1: ROW2 -> ROW3
- D14 pad 1: ROW3 -> ROW2
- D15 pad 1: ROW4 -> ROW1
- D17 pad 1: ROW2 -> ROW3
- D18 pad 1: ROW3 -> ROW2
- D19 pad 1: ROW4 -> ROW1
- D2 pad 1: ROW3 -> ROW2
- D21 pad 1: ROW2 -> ROW3
- D22 pad 1: ROW3 -> ROW2
- D23 pad 1: ROW4 -> ROW1
- D25 pad 1: ROW3 -> ROW2
- D26 pad 1: ROW4 -> ROW1
- D28 pad 1: ROW1 -> ROW4
- D29 pad 1: ROW1 -> ROW4
- D3 pad 1: ROW4 -> ROW1
- D30 pad 1: ROW1 -> ROW4
- D31 pad 1: ROW1 -> ROW4
- D32 pad 1: ROW1 -> ROW4
- D33 pad 1: ROW1 -> ROW4
- D34 pad 1: ROW1 -> ROW4
- D35 pad 1: ROW2 -> ROW3
- D5 pad 1: ROW2 -> ROW3
- D6 pad 1: ROW3 -> ROW2
- D7 pad 1: ROW4 -> ROW1
- D9 pad 1: ROW2 -> ROW3
- S1 pad 1: COL1 -> COL0
- S10 pad 1: COL3 -> COL2
- S11 pad 1: COL3 -> COL2
- S12 pad 1: COL3 -> COL2
- S13 pad 1: COL4 -> COL3
- S14 pad 1: COL4 -> COL3
- S15 pad 1: COL4 -> COL3
- S16 pad 1: COL4 -> COL3
- S17 pad 1: COL5 -> COL4
- S18 pad 1: COL5 -> COL4
- S19 pad 1: COL5 -> COL4
- S2 pad 1: COL1 -> COL0
- S20 pad 1: COL5 -> COL4
- S21 pad 1: COL6 -> COL5
- S22 pad 1: COL6 -> COL5
- S23 pad 1: COL6 -> COL5
- S24 pad 1: COL6 -> COL5
- S25 pad 1: COL7 -> COL6
- S26 pad 1: COL7 -> COL6
- S27 pad 1: COL7 -> COL6
- S28 pad 1: COL1 -> COL0
- S29 pad 1: COL2 -> COL1
- S3 pad 1: COL1 -> COL0
- S30 pad 1: COL3 -> COL2
- S31 pad 1: COL4 -> COL3
- S32 pad 1: COL5 -> COL4
- S33 pad 1: COL6 -> COL5
- S34 pad 1: COL7 -> COL6
- S35 pad 1: COL7 -> COL6
- S4 pad 1: COL1 -> COL0
- S5 pad 1: COL2 -> COL1
- S6 pad 1: COL2 -> COL1
- S7 pad 1: COL2 -> COL1
- S8 pad 1: COL2 -> COL1
- S9 pad 1: COL3 -> COL2
Other:
- outline, holes or cut-outs redrawn

Commit message: add more components to design data
Parts:
- added LED1: , WS2812B, F.Cu at (50.0, 95.3)
- added LED10: , WS2812B, F.Cu at (88.0, 71.5)
- added LED11: , WS2812B, F.Cu at (88.0, 52.4)
- added LED12: , WS2812B, F.Cu at (88.0, 33.4)
- added LED13: , WS2812B, F.Cu at (107.0, 88.2)
- added LED14: , WS2812B, F.Cu at (107.0, 69.1)
- added LED15: , WS2812B, F.Cu at (107.0, 50.1)
- added LED16: , WS2812B, F.Cu at (107.0, 31.0)
- added LED17: , WS2812B, F.Cu at (126.0, 90.5)
- added LED18: , WS2812B, F.Cu at (126.0, 71.5)
- added LED19: , WS2812B, F.Cu at (126.0, 52.4)
- added LED2: , WS2812B, F.Cu at (50.0, 76.2)
- added LED20: , WS2812B, F.Cu at (126.0, 33.4)
- added LED21: , WS2812B, F.Cu at (145.0, 92.9)
- added LED22: , WS2812B, F.Cu at (145.0, 73.9)
- added LED23: , WS2812B, F.Cu at (145.0, 54.8)
- added LED24: , WS2812B, F.Cu at (145.0, 35.8)
- added LED25: , WS2812B, F.Cu at (164.0, 83.4)
- added LED26: , WS2812B, F.Cu at (164.0, 64.3)
- added LED27: , WS2812B, F.Cu at (164.0, 45.3)
- added LED28: , WS2812B, F.Cu at (50.0, 114.3)
- added LED29: , WS2812B, F.Cu at (69.0, 114.3)
- added LED3: , WS2812B, F.Cu at (50.0, 57.2)
- added LED30: , WS2812B, F.Cu at (88.0, 109.6)
- added LED31: , WS2812B, F.Cu at (107.0, 107.2)
- added LED32: , WS2812B, F.Cu at (139.7, 116.4)
- added LED33: , WS2812B, F.Cu at (154.5, 119.4)
- added LED34: , WS2812B, F.Cu at (172.7, 135.5)
- added LED35: , WS2812B, F.Cu at (182.3, 119.0)
- added LED4: , WS2812B, F.Cu at (50.0, 38.2)
- added LED5: , WS2812B, F.Cu at (69.0, 95.3)
- added LED6: , WS2812B, F.Cu at (69.0, 76.2)
- added LED7: , WS2812B, F.Cu at (69.0, 57.2)
- added LED8: , WS2812B, F.Cu at (69.0, 38.2)
- added LED9: , WS2812B, F.Cu at (88.0, 90.5)
- turned S1 to 0 degrees
- turned S10 to 0 degrees
- turned S11 to 0 degrees
- turned S12 to 0 degrees
- turned S13 to 0 degrees
- turned S14 to 0 degrees
- turned S15 to 0 degrees
- turned S16 to 0 degrees
- turned S17 to 0 degrees
- turned S18 to 0 degrees
- turned S19 to 0 degrees
- turned S2 to 0 degrees
- turned S20 to 0 degrees
- turned S21 to 0 degrees
- turned S22 to 0 degrees
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